File: Schematics/EMS-ESP8266-12/EMS-ESP8266-12.sch (EAGLE design)
At the start: 44 parts, among them IC1 LM393N, T1 BC547B, T2 BC547B

Commit message: Attributes: add REICHELT order number and ALTERNATE package/part
Parts:
- C8: ALTERNATIV (none) -> SMD 10uF Keramik; REICHELT (none) -> X7R-G1206 10/16
- D1, D2, D3, D4: ALTERNATIV (none) -> 1/2 BAT54S
Changed lines of the file:
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@@
 <parts>
 <part name="D1" library="diode" deviceset="SCHOTTKY-DIODE" device="DO35-7" value="BAT46">
+<attribute name="ALTERNATIV" value="1/2 BAT54S"/>
 <attribute name="REICHELT" value="BAT 46"/>
 </part>
 <part name="D2" library="diode" deviceset="SCHOTTKY-DIODE" device="DO35-7" value="BAT46">
+<attribute name="ALTERNATIV" value="1/2 BAT54S"/>
 <attribute name="REICHELT" value="BAT 46"/>
 </part>
 <part name="D3" library="diode" deviceset="SCHOTTKY-DIODE" device="DO35-7" value="BAT46">
+<attribute name="ALTERNATIV" value="1/2 BAT54S"/>
 <attribute name="REICHELT" value="BAT 46"/>
 </part>
 <part name="D4" library="diode" deviceset="SCHOTTKY-DIODE" device="DO35-7" value="BAT46">
+<attribute name="ALTERNATIV" value="1/2 BAT54S"/>
 <attribute name="REICHELT" value="BAT 46"/>
 </part>
@@
 </part>
 <part name="C8" library="capacitor-wima" deviceset="C" device="5/11" value="10u">
+<attribute name="ALTERNATIV" value="SMD 10uF Keramik"/>
 <attribute name="CONRAD" value="450662-62"/>
+<attribute name="REICHELT" value="X7R-G1206 10/16"/>
 </part>
 <part name="C9" library="capacitor-wima" deviceset="C" device="2.5/2" value="1n">
@@
 <instance part="D1" gate="G$1" x="-137.16" y="175.26">
 <attribute name="REICHELT" x="-137.16" y="175.26" size="1.778" layer="96" display="off"/>
+<attribute name="ALTERNATIV" x="-137.16" y="175.26" size="1.778" layer="96" display="off"/>
 </instance>
 <instance part="D2" gate="G$1" x="-137.16" y="165.1" rot="R180">
 <attribute name="REICHELT" x="-137.16" y="165.1" size="1.778" layer="96" rot="R180" display="off"/>
+<attribute name="ALTERNATIV" x="-137.16" y="165.1" size="1.778" layer="96" rot="R180" display="off"/>
 </instance>
 <instance part="D3" gate="G$1" x="-137.16" y="152.4">
 <attribute name="REICHELT" x="-137.16" y="152.4" size="1.778" layer="96" display="off"/>
+<attribute name="ALTERNATIV" x="-137.16" y="152.4" size="1.778" layer="96" display="off"/>
 </instance>
 <instance part="D4" gate="G$1" x="-137.16" y="142.24" rot="R180">
 <attribute name="REICHELT" x="-137.16" y="142.24" size="1.778" layer="96" rot="R180" display="off"/>
+<attribute name="ALTERNATIV" x="-137.16" y="142.24" size="1.778" layer="96" rot="R180" display="off"/>
 </instance>
 <instance part="D5" gate="G$1" x="-127" y="147.32" rot="R90">
@@
 <instance part="C8" gate="G$1" x="-78.74" y="124.46" rot="R90">
 <attribute name="CONRAD" x="-78.74" y="124.46" size="1.778" layer="96" rot="R90" display="off"/>
+<attribute name="ALTERNATIV" x="-78.74" y="124.46" size="1.778" layer="96" rot="R90" display="off"/>
+<attribute name="REICHELT" x="-78.74" y="124.46" size="1.778" layer="96" rot="R90" display="off"/>
 </instance>
 <instance part="C9" gate="G$1" x="-78.74" y="119.38" rot="R90">
